File: teensy-breakout/teensy-breakout.kicad_pcb (KiCad board)
At the start: 6 copper layers, 240.5 x 168.5 mm, 158 parts, among them J1 USB_B, J10 1988820, J11 1988817, J12 1988817, J13 1988817, J14 1988817, J15 1988820, J16 1988956, J17 1988956, J18 1988817, J19 1989010, J2 1988820, J20 1989010, J21 1988956, J22 1988817, J3 1988820, J4 1988820, J5 1988820, J6 1988820, J7 1988820, J8 1988833, J9 1988956, Q1 IRL530NSTRLPBF, SW1 7101MD9AQE, U1 Teensy4.1, U10 LSF0102DCUR, U3 FT232RL, U6 ICL7667CBAZA-TDKR, U7 LSF0102DCUR, U8 LSF0102DCUR

Commit message: Did most of the routing, need to add pinouts and mounting holes
Parts:
- removed CR1, CR3, CR4: L7805CD2T-TR, Custom:D2PAKSMD_2L_STD-ST_STM
- removed R14: 200k, Resistor_SMD:R_0805_2012Metric_Pad1.20x1.40mm_HandSolder
- removed the REF** at (94.0, 109.2)
- removed the REF** at (220.1, 36.5)
- removed the REF** at (68.6, 119.4)
- removed the REF** at (86.4, 119.4)
- removed the REF** at (63.5, 119.4)
- removed the REF** at (149.5, 139.4)
- removed the REF** at (127.0, 179.1)
- removed the REF** at (78.7, 119.4)
- removed the REF** at (126.0, 189.8)
- removed the REF** at (50.8, 119.4)
- removed the REF** at (185.4, 114.3)
- removed the REF** at (48.2, 173.9)
- removed the REF** at (94.7, 92.7)
- removed the REF** at (167.6, 114.3)
- removed the REF** at (45.7, 119.4)
- removed the REF** at (165.1, 114.3)
- removed the REF** at (182.9, 114.3)
- removed the REF** at (193.0, 114.3)
- removed the REF** at (200.7, 114.3)
- removed the REF** at (133.9, 189.8)
- removed the REF** at (195.6, 114.3)
- removed the REF** at (71.1, 119.4)
- removed the REF** at (239.4, 158.3)
- removed the REF** at (197.9, 166.2)
- removed the REF** at (55.9, 119.4)
- removed the REF** at (188.0, 114.3)
- removed the REF** at (129.5, 175.3)
- removed the REF** at (160.0, 114.3)
- removed the REF** at (203.2, 114.3)
- removed the REF** at (177.6, 69.9)
- removed the REF** at (81.3, 119.4)
- removed the REF** at (96.5, 109.2)
- removed the REF** at (114.3, 264.2)
- removed the REF** at (142.0, 101.5)
- removed the REF** at (83.8, 205.7)
- removed the REF** at (177.6, 101.3)
- removed the REF** at (120.1, 147.1)
- removed the REF** at (48.3, 119.4)
- removed the REF** at (88.9, 119.4)
- removed the REF** at (133.9, 147.2)
- removed the REF** at (127.0, 175.3)
- removed the REF** at (143.4, 82.0)
- removed the REF** at (154.9, 114.3)
- removed the REF** at (165.0, 170.1)
- removed the REF** at (38.1, 119.4)
- removed the REF** at (205.7, 114.3)
- removed the REF** at (83.8, 119.4)
- removed the REF** at (43.2, 119.4)
- removed the REF** at (152.4, 114.3)
- removed the REF** at (170.2, 114.3)
- removed the REF** at (36.4, 162.7)
- removed the REF** at (171.4, 140.7)
- removed the REF** at (79.4, 147.0)
- removed the REF** at (66.0, 119.4)
- removed the REF** at (50.2, 32.3)
- removed the REF** at (73.7, 119.4)
- removed the REF** at (124.0, 84.9)
- removed the REF** at (58.4, 119.4)
- removed the REF** at (144.3, 72.7)
- removed the REF** at (172.7, 114.3)
- removed the REF** at (99.0, 30.3)
- removed the REF** at (198.1, 114.3)
- removed the REF** at (180.3, 114.3)
- removed the REF** at (149.9, 114.3)
- removed the REF** at (162.6, 114.3)
- removed the REF** at (91.4, 119.4)
- removed the REF** at (165.1, 190.7)
- removed the REF** at (53.3, 119.4)
- removed the REF** at (40.6, 119.4)
- removed the REF** at (177.8, 114.3)
- removed the REF** at (76.2, 119.4)
- removed the REF** at (175.3, 114.3)
- removed the REF** at (157.5, 114.3)
- removed the REF** at (61.0, 119.4)
- removed the REF** at (147.3, 114.3)
- removed the REF** at (190.5, 114.3)
- removed U8: LSF0102DCUR, Custom:DCU0008A_M
- added REF**: PinHeader_1x24_P2.54mm_Vertical, Connector_PinHeader_2.54mm:PinHeader_1x24_P2.54mm_Vertical, F.Cu at (182.9, 138.4)
- added REF**: PinHeader_1x24_P2.54mm_Vertical, Connector_PinHeader_2.54mm:PinHeader_1x24_P2.54mm_Vertical, F.Cu at (154.9, 138.4)
- added U9: ~, Custom:Pololu D36V50F5, F.Cu at (122.0, 216.0)
- J10, J15, J4, J5, J6, J7: value 1988820 -> Conn_01x04; footprint Custom:CONN_1988820 -> Connector_JST:JST_EH_B4B-EH-A_1x04_P2.50mm_Vertical
- J11, J14: value 1988817 -> Conn_01x04; footprint Custom:CONN_1988817 -> Connector_JST:JST_EH_B4B-EH-A_1x04_P2.50mm_Vertical
- J12: value 1988817 -> Conn_01x05; footprint Custom:CONN_1988817 -> Connector_JST:JST_EH_B5B-EH-A_1x05_P2.50mm_Vertical
- J13, J22: value 1988817 -> Conn_01x03; footprint Custom:CONN_1988817 -> Connector_JST:JST_EH_B3B-EH-A_1x03_P2.50mm_Vertical
- J16: value 1988956 -> Conn_01x02; footprint Custom:CONN_1988956 -> Connector_JST:JST_EH_B2B-EH-A_1x02_P2.50mm_Vertical
- J17: value 1988956 -> Conn_01x08; footprint Custom:CONN_1988956 -> Custom:PHOENIX_1989010
- J18: value 1988817 -> Conn_01x08; footprint Custom:CONN_1988817 -> Custom:PHOENIX_1989010
- J19, J20: value 1989010 -> Conn_01x03; footprint Custom:PHOENIX_1989010 -> Connector_JST:JST_EH_B3B-EH-A_1x03_P2.50mm_Vertical
- J2, J3: value 1988820 -> Conn_01x02; footprint Custom:CONN_1988820 -> Connector_AMASS:AMASS_XT60-F_1x02_P7.20mm_Vertical
- J21: value 1988956 -> Conn_01x03; footprint Custom:CONN_1988956 -> Connector_JST:JST_EH_B3B-EH-A_1x03_P2.50mm_Vertical
- J8: value 1988833 -> Conn_01x04; footprint Custom:CONN_1988833 -> Connector_JST:JST_EH_B4B-EH-A_1x04_P2.50mm_Vertical
- J9: value 1988956 -> Conn_01x04; footprint Custom:CONN_1988956 -> Connector_JST:JST_EH_B4B-EH-A_1x04_P2.50mm_Vertical
- Q1: footprint Custom:D2PAKSMD_2L_STD-ST_STM -> Custom:IRL530NSTRLPBF_INF
- moved J10 250.6 mm to (195.7, 221.0), turned to 0 degrees
- moved R10 248.3 mm to (182.9, 246.4), turned to 90 degrees
- moved R9 241.1 mm to (180.3, 246.4), turned to 90 degrees
- moved J5 240.4 mm to (210.9, 255.3), turned to 0 degrees
- moved J11 235.8 mm to (188.0, 241.0)
- moved J9 222.6 mm to (180.3, 255.3), turned to 0 degrees
- moved Q1 217.0 mm to (120.7, 251.1), turned to 180 degrees
- moved J2 215.2 mm to (133.8, 236.2), turned to 0 degrees
- moved J17 207.6 mm to (238.0, 238.9)
- moved J7 203.7 mm to (195.7, 255.3), turned to 0 degrees
- moved J6 203.3 mm to (149.9, 255.3), turned to 0 degrees
- moved J15 199.8 mm to (156.1, 204.5)
- moved J21 198.1 mm to (186.7, 227.3)
- moved CR2 197.8 mm to (111.8, 249.5), turned to 180 degrees
- moved R2 193.3 mm to (125.7, 242.5), turned to 90 degrees
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Connections:
- J10 pad 1: GND -> +5V
- J10 pad 2: GND -> /RC_RX
- J10 pad 3: /LIM_R -> /RC_TX
- J10 pad 4: /LIM_L -> GND
- J11 pad 1: Net-(CR4-OUTPUT) -> GND
- J11 pad 2: Net-(U10-B1) -> GND
- J11 pad 3: GND -> /LIM_R
- J12 pad 1: Net-(CR4-OUTPUT) -> /ALM
- J12 pad 2: Net-(U10-B2) -> /DIR_MIN
- J12 pad 3: GND -> /PUL_MIN
- J13 pad 1: Net-(CR4-OUTPUT) -> /I2C1_SDA
- J13 pad 2: Net-(U7-B1) -> /I2C1_SCL
- J14 pad 1: Net-(CR4-OUTPUT) -> /MOSI0
- J14 pad 2: Net-(U7-B2) -> /MISO0
- J14 pad 3: GND -> /SCK0
- J15 pad 1: +5V -> /MOSI1
- J15 pad 2: Net-(U8-B1) -> /MISO1
- J15 pad 3: Net-(U8-B2) -> /SCK1
- J17 pad 1: Net-(U1-17_A3_TX4_SDA1) -> /J1_1
- J17 pad 2: Net-(U1-16_A2_RX4_SCL1) -> /J1_2
- J18 pad 1: /MOSI0 -> /J0_1
- J18 pad 2: /MISO0 -> /J0_2
- J18 pad 3: /SCK0 -> /J0_3
- J19 pad 1: /J0_1 -> +5V
- J19 pad 2: /J0_2 -> /NP1_5V
- J19 pad 3: /J0_3 -> GND
- J2 pad 1: GND -> Net-(J2-Pin_1)
- J20 pad 1: /J1_1 -> +5V
- J20 pad 2: /J1_2 -> /NP2_5V
- J20 pad 3: /J1_3 -> GND
- J21 pad 1: +12V -> +5V
- J21 pad 2: GND -> /NP3_5V
- J22 pad 1: /MOSI1 -> +5V
- J22 pad 2: /MISO1 -> /NP4_5V
- J22 pad 3: /SCK1 -> GND
- J3 pad 1: GND -> Net-(D3-K)
- J3 pad 2: GND -> +12V
- J4 pad 1: +3V3 -> GND
- J4 pad 2: +3V3 -> GND
- J4 pad 3: +3V3 -> GND
- J4 pad 4: +3V3 -> GND
- J5 pad 1: +3V3 -> GND
- J5 pad 2: +3V3 -> GND
- J5 pad 3: +3V3 -> GND
- J5 pad 4: +3V3 -> GND
- J6 pad 1: Net-(CR3-OUTPUT) -> +3V3
- J6 pad 2: Net-(CR3-OUTPUT) -> +3V3
- J6 pad 3: Net-(CR3-OUTPUT) -> +3V3
- J6 pad 4: Net-(CR3-OUTPUT) -> +3V3
- J7 pad 1: Net-(CR3-OUTPUT) -> +3V3
- J7 pad 2: Net-(CR3-OUTPUT) -> +3V3
- J7 pad 3: Net-(CR3-OUTPUT) -> +3V3
- J7 pad 4: Net-(CR3-OUTPUT) -> +3V3
- J8 pad 1: /ALM -> +5V
- J8 pad 2: /DIR_MIN -> +5V
- J8 pad 3: /PUL_MIN -> +5V
- J9 pad 1: Net-(D3-K) -> +5V
- J9 pad 2: +12V -> +5V
- R11 pad 2: Net-(U1-17_A3_TX4_SDA1) -> /I2C1_SDA
- R12 pad 2: Net-(U1-16_A2_RX4_SCL1) -> /I2C1_SCL
- R15 pad 1: Net-(CR4-OUTPUT) -> +5V
- R16 pad 1: Net-(CR4-OUTPUT) -> +5V
- U1 pad 38: Net-(U1-16_A2_RX4_SCL1) -> /I2C1_SCL
- U1 pad 39: Net-(U1-17_A3_TX4_SDA1) -> /I2C1_SDA
- U10 pad 5: Net-(U10-B2) -> /NP2_5V
- U10 pad 6: Net-(U10-B1) -> /NP1_5V
- U7 pad 5: Net-(U7-B2) -> /NP4_5V
- U7 pad 6: Net-(U7-B1) -> /NP3_5V
Routing:
- net GND: track 0.00 -> 194.1 mm, vias 0 -> 6
- net /I2C0_SCL: track 0.00 -> 151.5 mm
- net /I2C0_SDA: track 0.00 -> 146.6 mm, vias 0 -> 1
- net /PUL: track 0.00 -> 136.1 mm, vias 0 -> 3
- net /BRAKE: track 0.00 -> 126.5 mm, vias 0 -> 3
- net /J1_7: track 0.00 -> 116.7 mm
- net /ALM: track 0.00 -> 107.6 mm, vias 0 -> 2
- net /J0_6: track 0.00 -> 107.2 mm, vias 0 -> 1
- net /SCK0: track 0.00 -> 91.2 mm
- net /J1_6: track 0.00 -> 89.6 mm
- net +3V3: track 0.00 -> 89.1 mm, vias 0 -> 3
- net +5V: track 0.00 -> 88.5 mm, vias 0 -> 3
- net /J1_5: track 0.00 -> 88.2 mm, vias 0 -> 1
- net /NP3: track 0.00 -> 86.5 mm, vias 0 -> 1
- net /RC_RX: track 0.00 -> 85.3 mm, vias 0 -> 1
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- added copper zone on In4.Cu, net +12V
- added copper zone on In3.Cu, net +5V
- removed copper zone on In3.Cu, net +12V
- removed copper zone on In4.Cu, net +5V
Other:
- board size 240.5 x 168.5 mm -> 139.7 x 133.4 mm
- board text removed: "+12V"
- board text removed: "+3V3"
- board text removed: "+3V3 GPIO"
- board text removed: "+5V"
- board text removed: "+5V GPIO"
- board text removed: "0"
- board text removed: "1"
- board text removed: "10"
- board text removed: "11"
- board text removed: "12"
- board text removed: "13"
- board text removed: "14"
- board text removed: "15"
- board text removed: "16"
- board text removed: "17"
- board text removed: "18"
- board text removed: "19"
- board text removed: "2"
- board text removed: "20"
- board text removed: "21"
- board text removed: "22"
- board text removed: "23"
- board text removed: "24"
- board text removed: "25"
- board text removed: "26"
- board text removed: "27"
- board text removed: "28"
- board text removed: "29"
- board text removed: "3"
- board text removed: "30"
- board text removed: "31"
- board text removed: "32"
- board text removed: "33"
- board text removed: "34"
- board text removed: "35"
- board text removed: "36"
- board text removed: "37"
- board text removed: "38"
- board text removed: "39"
- board text removed: "4"
- board text removed: "40"
- board text removed: "41"
- board text removed: "5"
- board text removed: "6"
- board text removed: "7"
- board text removed: "8"
- board text removed: "9"
- board text removed: "ALM"
- board text removed: "BRAKE SOLENOID"
- board text removed: "Bank 0"
- board text removed: "Bank 1"
- board text removed: "Brake LED"
- board text removed: "CS"
- board text removed: "DIR_MIN"
- board text removed: "DIR_PLUS"
- board text removed: "G0"
- board text removed: "GND"
- board text removed: "GPS Serial"
- board text removed: "I2C0"
- board text removed: "I2C1"
- board text removed: "L"
- board text removed: "LIMIT SWITCHES"
- board text removed: "MISO0"
- board text removed: "MISO1"
- board text removed: "MOSI0"
- board text removed: "MOSI1"
- board text removed: "NC"
- board text removed: "OUT"
- board text removed: "POWER INPUT"
- board text removed: "POWER SWITCH"
- board text removed: "PUL_MIN"
- board text removed: "PUL_PLUS"
- board text removed: "Power from CR3 linear regulator"
- board text removed: "Power from CR4 linear regulator"
- board text removed: "R"
- board text removed: "RC STATION"
- board text removed: "RST"
- board text removed: "RX"
- board text removed: "SCK0"
- board text removed: "SCK1"
- board text removed: "SCL"
- board text removed: "SCL1"
- board text removed: "SDA"
- board text removed: "SDA1"
- board text removed: "SPI0"
- board text removed: "SPI1"
- board text removed: "STEPPER CONTROL"
- board text removed: "TEENSY_RX"
- board text removed: "TEENSY_TX"
- board text removed: "TX"
